File: schematics/buttonRelayModuleControl/buttonRelayModuleControl.kicad_pcb (KiCad board)
At the start: 2 copper layers, 73.2 x 42.2 mm, 23 parts, among them J1 Conn_AC_MAINS, J2 Programmer, SW1 SW_Push_LED, SW2 SW_Push_LED, U1 HLK-5M05, U3 ATmega328PB-AU

Commit message: Add logo to board
Parts:
- added G***: LOGO, ml_logo:ML_Logo, B.Cu at (154.2, 89.9)
Other:
- board text added: "2 Channel Float Swtich"
Changed lines of the file:
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@@
   (general
     (thickness 1.6)
-    (drawings 4)
+    (drawings 5)
     (tracks 162)
     (zones 0)
-    (modules 23)
+    (modules 24)
     (nets 37)
   )
@@
       (padsonsilk false)
       (subtractmaskfromsilk false)
-      (outputformat 1)
+      (outputformat 5)
       (mirror false)
-      (drillshape 1)
+      (drillshape 0)
       (scaleselection 1)
-      (outputdirectory ""))
+      (outputdirectory "./board.svg"))
   )
   (net 0 "")
@@
     )
   )
+  (module ml_logo:ML_Logo (layer B.Cu)
+    (at 154.178 89.916 180)
+    (attr smd)
+    (fp_text reference G*** (at 0 0 180) (layer B.SilkS) hide
+      (effects (font (size 1.524 1.524) (thickness 0.3)) (justify mirror))
+    )
+    (fp_text value LOGO (at 0.75 0 180) (layer B.SilkS) hide
+      (effects (font (size 1.524 1.524) (thickness 0.3)) (justify mirror))
+    )
+    (fp_poly (pts (xy 1.453015 3.880254) (xy 1.486479 3.418381) (xy 1.411872 2.664402) (xy 1.230095 1.631252)
+      (xy 1.100201 1.018098) (xy 0.927611 -0.109332) (xy 0.966577 -0.97695) (xy 1.21686 -1.584098)
+      (xy 1.678216 -1.930119) (xy 2.214865 -2.018543) (xy 2.58487 -1.949839) (xy 3.145836 -1.768138)
+      (xy 3.787397 -1.510056) (xy 3.901609 -1.458913) (xy 4.76076 -1.095062) (xy 5.456136 -0.855597)
+      (xy 5.9488 -0.75072) (xy 6.199814 -0.790631) (xy 6.223842 -0.850544) (xy 6.086782 -1.040256)
+      (xy 5.929471 -1.120354) (xy 5.652766 -1.228084) (xy 5.151615 -1.43478) (xy 4.510178 -1.705463)
+      (xy 4.120899 -1.872028) (xy 3.039497 -2.283428) (xy 2.184746 -2.484242) (xy 1.524917 -2.47934)
+      (xy 1.11967 -2.332673) (xy 0.783673 -1.978373) (xy 0.51366 -1.403055) (xy 0.355945 -0.721551)
+      (xy 0.333692 -0.38388) (xy 0.364747 0.041488) (xy 0.450911 0.698507) (xy 0.578113 1.489593)
+      (xy 0.698276 2.144702) (xy 0.884526 3.033718) (xy 1.042856 3.622655) (xy 1.184292 3.945595)
+      (xy 1.310579 4.037086) (xy 1.453015 3.880254)) (layer B.SilkS) (width 0.01))
+    (fp_poly (pts (xy -0.447799 4.677159) (xy -0.350536 4.551497) (xy -0.277038 4.291944) (xy -0.22199 3.857495)
+      (xy -0.180079 3.207146) (xy -0.145991 2.299892) (xy -0.116364 1.177483) (xy -0.086755 0.226168)
+      (xy -0.047148 -0.621582) (xy -0.001542 -1.302222) (xy 0.046066 -1.752205) (xy 0.076817 -1.892384)
+      (xy 0.1137 -2.132539) (xy 0.044998 -2.186755) (xy -0.183918 -2.021975) (xy -0.372225 -1.537226)
+      (xy -0.51656 -0.746893) (xy -0.613563 0.334636) (xy -0.632983 0.7149) (xy -0.675531 1.48523)
+      (xy -0.727483 2.115182) (xy -0.782218 2.539105) (xy -0.832349 2.691391) (xy -0.933714 2.543351)
+      (xy -1.07226 2.163236) (xy -1.165679 1.83296) (xy -1.375501 1.172042) (xy -1.667109 0.456141)
+      (xy -2.001167 -0.238347) (xy -2.338337 -0.835025) (xy -2.639282 -1.257497) (xy -2.842996 -1.424531)
+      (xy -3.244705 -1.456647) (xy -3.416895 -1.418594) (xy -3.735704 -1.155621) (xy -4.056408 -0.66466)
+      (xy -4.321367 -0.048837) (xy -4.4474 0.425236) (xy -4.533679 0.776758) (xy -4.623136 0.893202)
+      (xy -4.722196 0.755938) (xy -4.837284 0.346336) (xy -4.974827 -0.354234) (xy -5.141247 -1.364402)
+      (xy -5.203195 -1.766225) (xy -5.339266 -2.648673) (xy -5.463959 -3.43734) (xy -5.565581 -4.059669)
+      (xy -5.632437 -4.443101) (xy -5.643744 -4.499669) (xy -5.79234 -4.766295) (xy -6.014664 -4.879658)
+      (xy -6.190763 -4.805012) (xy -6.224476 -4.667881) (xy -6.193656 -4.407975) (xy -6.104516 -3.85109)
+      (xy -5.96294 -3.030483) (xy -5.774815 -1.979416) (xy -5.546027 -0.731148) (xy -5.282461 0.681061)
+      (xy -5.207727 1.077535) (xy -5.057832 1.799753) (xy -4.907751 2.402058) (xy -4.778845 2.804213)
+      (xy -4.717365 2.919455) (xy -4.489736 3.008993) (xy -4.300316 2.7791) (xy -4.14678 2.224546)
+      (xy -4.030013 1.372216) (xy -3.921272 0.5106) (xy -3.783506 -0.089719) (xy -3.59174 -0.503843)
+      (xy -3.320996 -0.806872) (xy -3.299232 -0.825208) (xy -3.051155 -0.855484) (xy -2.758481 -0.56816)
+      (xy -2.419318 0.040278) (xy -2.031774 0.973346) (xy -1.593955 2.234559) (xy -1.5086 2.500036)
+      (xy -1.177243 3.48848) (xy -0.902625 4.196369) (xy -0.691852 4.606899) (xy -0.57414 4.709934)
+      (xy -0.447799 4.677159)) (layer B.SilkS) (width 0.01))
+  )
+  (gr_text "2 Channel \nFloat Swtich" (at 151.638 96.52) (layer B.SilkS)
+    (effects (font (size 1.5 1.5) (thickness 0.3)) (justify mirror))
+  )
   (gr_line (start 102.616 73.406) (end 175.768 73.406) (layer Edge.Cuts) (width 0.1))
